File: PCB/hackpad.kicad_sch (KiCad schematic)
At the start: 13 parts, among them SW1 SW_Push, SW2 SW_Push, SW3 SW_Push, SW4 SW_Push, SW5 SW_Push, SW6 SW_Push, U1 XIAO-RP2040-DIP

Commit message: demo
Connections:
- net GND: now also D3.2 (VSS)
Changed lines of the file:
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@@
+	(wire
+		(pts
+			(xy 186.69 54.61) (xy 213.36 54.61)
+		)
+		(stroke
+			(width 0)
+			(type default)
+		)
+	)
 	(wire
 		(pts
